File: eagle/dueSkel.brd (EAGLE design)
At the start: 88.1 x 58.4 mm, 36 parts, among them J13 FEMALE 2x3

Commit message: cleg boards
Routing:
- net D20: track 43.8 -> 41.3 mm
- net D19: track 13.7 -> 12.6 mm
- net N$12: track 3.05 -> 3.89 mm
- net N$9: track 3.05 -> 3.89 mm
- net D17: track 28.4 -> 27.6 mm
- net D10: track 16.0 -> 16.7 mm
- net N$6: track 3.05 -> 3.65 mm
